Commit message: add imu sensor and gps sensor to the simulation file

File: src/scout_2/urdf/empty.urdf (robot description, URDF)
Before this commit: robot None, 1 links, 1 joints
Links:
- added link gps_link
- added link imu_sensor_link; visual mesh filename=file:///home/marco/4d_thesis/src/scout_2/meshes/laser_link.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 scale=1.5 1.5 1.5
Joints:
- added joint gps_sensor: type fixed, parent chassis_link, child gps_link, origin xyz=0.0 0.0 0.40 rpy=0 0 0
- added joint imu_sensor: type fixed, parent chassis_link, child imu_sensor_link, origin xyz=0.0 0.0 0.50 rpy=0 0 0

Commit message: add a new world and the usage of mapviz. written other launch file to launch this new world together with the ekf_localization and a new nav2 params file without the static glocal costmap

File: src/scout_2/urdf/empty.urdf (robot description, URDF)
Before this commit: robot None, 3 links, 3 joints
Joints:
- joint gps_sensor: parent chassis_link -> base_link
- joint imu_sensor: parent chassis_link -> base_link
- joint os_sensor: parent chassis_link -> base_link

File: src/scout_2/urdf/scout.urdf (robot description, URDF)
Before this commit: robot scout_description, 8 links, 7 joints
Links:
- removed link base_footprint
- removed link inertial_link
- added link chassis_link, mass 40; collision box size=0.9250000 0.380000 0.210000; visual mesh filename=file:///home/marco/4d_thesis/src/scout_2/meshes/base_link.d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
- added link gps_link
- added link imu_sensor_link; visual mesh filename=file:///home/marco/4d_thesis/src/scout_2/meshes/laser_link.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 scale=1.5 1.5 1.5
- link base_link: geometry 
- link os_sensor_link: geometry visual mesh filename=file:///home/marco/4d_thesis/src/scout_2/meshes/os1_64.stl scale=1.5 1.5 1.5
Joints:
- removed joint base_footprint_joint
- removed joint inertial_joint
- added joint chassis_joint: type fixed, parent base_link, child chassis_link, origin xyz=0 0 -0.23479 rpy=0 0 0
- added joint gps_sensor: type fixed, parent chassis_link, child gps_link, origin xyz=0.0 0.0 0.40 rpy=0 0 0
- added joint imu_sensor: type fixed, parent chassis_link, child imu_sensor_link, origin xyz=0.0 0.0 0.50 rpy=0 0 0
- joint front_left_wheel: axis 0 1 0 -> 0 0 1; limit effort=1000 velocity=1.5 -> effort=200 velocity=1.5; origin xyz=0.249 0.29153 -0.0702 rpy=0 0 0 -> xyz=0.249 0.29153 -0.0702 rpy=-1.570795 0 0; parent base_link -> chassis_link
- joint front_right_wheel: axis 0 1 0 -> 0 0 -1; limit effort=1000 velocity=1.5 -> effort=200 velocity=1.5; origin xyz=0.249 -0.29153 -0.0702 rpy=3.14 0 0 -> xyz=0.249 -0.29153 -0.0702 rpy=1.570795 0 0; parent base_link -> chassis_link
- joint os_sensor: parent base_link -> chassis_link
- joint rear_left_wheel: axis 0 1 0 -> 0 0 1; limit effort=1000 velocity=1.5 -> effort=200 velocity=1.5; origin xyz=-0.249 0.29153 -0.0702 rpy=0 0 0 -> xyz=-0.249 0.29153 -0.0702 rpy=-1.570795 0 0; parent base_link -> chassis_link
- joint rear_right_wheel: axis 0 1 0 -> 0 0 -1; limit effort=1000 velocity=1.5 -> effort=200 velocity=1.5; origin xyz=-0.249 -0.29153 -0.0702 rpy=3.14 0 0 -> xyz=-0.249 -0.29153 -0.0702 rpy=1.570795 0 0; parent base_link -> chassis_link

File: src/scout_2/urdf/scout_prova.xacro (robot description, xacro)
@@ -16,13 +16,12 @@
     <xacro:property name="wheel_radius" value="1.6459e-01" />
     <!-- Base link -->
-    <link name= "base_link">
-    </link>
+    <link name= "base_footprint"/>
     <!-- Chassis link -->
     <joint name="chassis_joint" type="fixed">
         <origin xyz="0 0 0.23479" rpy="0 0 0" />
-        <parent link="base_link" />
-        <child link="chassis_link" />
+        <parent link="base_footprint" />
+        <child link="base_link" />
     </joint>
-    <link name="chassis_link">
+    <link name="base_link">
         <visual>
             <origin xyz="0 0 0" rpy="0 0 0" />
@@ -69,5 +68,5 @@
     </link>
     <joint name="front_right_wheel" type="continuous">
-        <parent link="chassis_link"/>
+        <parent link="base_link"/>
         <child link="front_right_wheel_link"/>
         <origin rpy="1.570795 0 0" xyz="0.249 -0.29153 -0.0702"/>
@@ -101,5 +100,5 @@
     </link>
     <joint name="front_left_wheel" type="continuous">
-        <parent link="chassis_link"/>
+        <parent link="base_link"/>
         <child link="front_left_wheel_link"/>
         <origin rpy="-1.570795 0 0" xyz="0.249 0.29153 -0.0702"/>
@@ -133,5 +132,5 @@
     </link>
     <joint name="rear_left_wheel" type="continuous">
-        <parent link="chassis_link"/>
+        <parent link="base_link"/>
         <child link="rear_left_wheel_link"/>
         <origin rpy="-1.570795 0 0" xyz="-0.249 0.29153 -0.0702"/>
@@ -165,5 +164,5 @@
     </link>
     <joint name="rear_right_wheel" type="continuous">
-        <parent link="chassis_link"/>
+        <parent link="base_link"/>
         <child link="rear_right_wheel_link"/>
         <origin rpy="1.570795 0 0" xyz="-0.249 -0.29153 -0.0702"/>

Commit message: removed GPS IMU, now the EKF localize without GPS but with an odometry provided by the lidar thanks to the node lida_odometry

File: src/scout_2/urdf/empty.urdf (robot description, URDF)
Before this commit: robot None, 3 links, 3 joints
Links:
- removed link gps_link
- removed link imu_sensor_link
Joints:
- removed joint gps_sensor
- removed joint imu_sensor

Commit message: insert a node for converting lidar into odometry and correct the code

File: src/scout_2/urdf/empty.urdf (robot description, URDF)
Before this commit: robot None, 1 links, 1 joints
Joints:
- joint os_sensor: origin xyz=0.1 0.0 0.714 rpy=0 0 0 -> xyz=0.0 0.0 0.5 rpy=0 0 0

Commit message: final version of the project

File: src/scout_2/urdf/empty.urdf (robot description, URDF)
Before this commit: robot None, 1 links, 1 joints
Joints:
- joint os_sensor: origin xyz=0.0 0.0 0.5 rpy=0 0 0 -> xyz=0.0 0.0 0.2 rpy=0 0 0
